File: Output_HMC900.sch (KiCad schematic (older format))
At the start: 5 parts

Commit message: Corrected errors from single ended transition
Changed lines of the file:
@@
 $Descr A4 11693 8268
 encoding utf-8
-Sheet 3 7
+Sheet 6 7
 Title ""
 Date ""
@@
 AR Path="/60D21B6E/615E1BD1/614E552D" Ref="R?"  Part="1"
 AR Path="/60D21B6E/6160D475/614E552D" Ref="R16"  Part="1"
-AR Path="/60D21B6E/60F5ADAC/614E552D" Ref="R?"  Part="1"
-F 0 "R?" H 5980 3254 50  0000 R CNN
+AR Path="/60D21B6E/60F5ADAC/614E552D" Ref="R16"  Part="1"
+F 0 "R16" H 5980 3254 50  0000 R CNN
 F 1 "140" H 5980 3345 50  0000 R CNN
 F 2 "Resistor_SMD:R_0402_1005Metric" V 5980 3300 50  0001 C CNN
@@
 AR Path="/60D21B6E/615E1BD1/614E5533" Ref="R?"  Part="1"
 AR Path="/60D21B6E/6160D475/614E5533" Ref="R24"  Part="1"
-AR Path="/60D21B6E/60F5ADAC/614E5533" Ref="R?"  Part="1"
-F 0 "R?" V 5650 2950 50  0000 C CNN
+AR Path="/60D21B6E/60F5ADAC/614E5533" Ref="R15"  Part="1"
+F 0 "R15" V 5650 2950 50  0000 C CNN
 F 1 "174" V 5750 2950 50  0000 C CNN
 F 2 "Resistor_SMD:R_0402_1005Metric" V 5680 2950 50  0001 C CNN
@@
 AR Path="/60D21B6E/615E1BD1/614E5539" Ref="C?"  Part="1"
 AR Path="/60D21B6E/6160D475/614E5539" Ref="C43"  Part="1"
-AR Path="/60D21B6E/60F5ADAC/614E5539" Ref="C?"  Part="1"
-F 0 "C?" H 6465 3446 50  0000 L CNN
+AR Path="/60D21B6E/60F5ADAC/614E5539" Ref="C43"  Part="1"
+F 0 "C43" H 6465 3446 50  0000 L CNN
 F 1 "10u" H 6465 3355 50  0000 L CNN
 F 2 "Capacitor_SMD:C_0402_1005Metric" H 6388 3250 50  0001 C CNN
@@
 AR Path="/60D21B6E/615E1BD1/614E557C" Ref="#PWR?"  Part="1"
 AR Path="/60D21B6E/6160D475/614E557C" Ref="#PWR0140"  Part="1"
-AR Path="/60D21B6E/60F5ADAC/614E557C" Ref="#PWR?"  Part="1"
-F 0 "#PWR?" H 6350 3400 50  0001 C CNN
+AR Path="/60D21B6E/60F5ADAC/614E557C" Ref="#PWR0139"  Part="1"
+F 0 "#PWR0139" H 6350 3400 50  0001 C CNN
 F 1 "GND" H 6355 3477 50  0000 C CNN
 F 2 "" H 6350 3650 50  0001 C CNN
@@
 AR Path="/60D21B6E/615E1BD1/614E55C8" Ref="R?"  Part="1"
 AR Path="/60D21B6E/6160D475/614E55C8" Ref="R15"  Part="1"
-AR Path="/60D21B6E/60F5ADAC/614E55C8" Ref="R?"  Part="1"
-F 0 "R?" V 5650 3650 50  0000 C CNN
+AR Path="/60D21B6E/60F5ADAC/614E55C8" Ref="R24"  Part="1"
+F 0 "R24" V 5650 3650 50  0000 C CNN
 F 1 "174" V 5750 3650 50  0000 C CNN
 F 2 "Resistor_SMD:R_0402_1005Metric" V 5680 3650 50  0001 C CNN
@@
 AR Path="/60D21B6E/615E1BD1/614E5583" Ref="#PWR?"  Part="1"
 AR Path="/60D21B6E/6160D475/614E5583" Ref="#PWR0142"  Part="1"
-AR Path="/60D21B6E/60F5ADAC/614E5583" Ref="#PWR?"  Part="1"
-F 0 "#PWR?" H 7500 3200 50  0001 C CNN
+AR Path="/60D21B6E/60F5ADAC/614E5583" Ref="#PWR0140"  Part="1"
+F 0 "#PWR0140" H 7500 3200 50  0001 C CNN
 F 1 "GND" H 7505 3277 50  0000 C CNN
 F 2 "" H 7500 3450 50  0001 C CNN
@@
 AR Path="/60D21B6E/615E1BD1/614E5545" Ref="TR?"  Part="1"
 AR Path="/60D21B6E/6160D475/614E5545" Ref="TR2"  Part="1"
-AR Path="/60D21B6E/60F5ADAC/614E5545" Ref="TR?"  Part="1"
-F 0 "TR?" H 7150 3581 50  0000 C CNN
+AR Path="/60D21B6E/60F5ADAC/614E5545" Ref="TR2"  Part="1"
+F 0 "TR2" H 7150 3581 50  0000 C CNN
 F 1 "ADT2-1T" H 7150 3490 50  0000 C CNN
 F 2 "RF_Mini-Circuits:Mini-Circuits_CD542_H2.84mm" H 7150 2850 50  0001 C CNN

Commit message: passage 0402 => 0603
Parts:
- C44: footprint Capacitor_SMD:C_0402_1005Metric -> Capacitor_SMD:C_0603_1608Metric_Pad1.08x0.95mm_HandSolder
- R11, R12, R21: footprint Resistor_SMD:R_0402_1005Metric -> Resistor_SMD:R_0603_1608Metric_Pad0.98x0.95mm_HandSolder
Changed lines of the file:
@@
 $Descr A4 11693 8268
 encoding utf-8
-Sheet 6 7
+Sheet 3 7
 Title ""
 Date ""
@@
 AR Path="/60D21B6E/6160D475/614E552D" Ref="R16"  Part="1"
 AR Path="/60D21B6E/60F5ADAC/614E552D" Ref="R16"  Part="1"
-F 0 "R16" H 5980 3254 50  0000 R CNN
+F 0 "R11" H 5980 3254 50  0000 R CNN
 F 1 "140" H 5980 3345 50  0000 R CNN
-F 2 "Resistor_SMD:R_0402_1005Metric" V 5980 3300 50  0001 C CNN
+F 2 "Resistor_SMD:R_0603_1608Metric_Pad0.98x0.95mm_HandSolder" V 5980 3300 50  0001 C CNN
 F 3 "~" H 6050 3300 50  0001 C CNN
 	1    6050 3300
@@
 AR Path="/60D21B6E/6160D475/614E5533" Ref="R24"  Part="1"
 AR Path="/60D21B6E/60F5ADAC/614E5533" Ref="R15"  Part="1"
-F 0 "R15" V 5650 2950 50  0000 C CNN
+F 0 "R21" V 5650 2950 50  0000 C CNN
 F 1 "174" V 5750 2950 50  0000 C CNN
-F 2 "Resistor_SMD:R_0402_1005Metric" V 5680 2950 50  0001 C CNN
+F 2 "Resistor_SMD:R_0603_1608Metric_Pad0.98x0.95mm_HandSolder" V 5680 2950 50  0001 C CNN
 F 3 "~" H 5750 2950 50  0001 C CNN
 	1    5750 2950
@@
 AR Path="/60D21B6E/6160D475/614E5539" Ref="C43"  Part="1"
 AR Path="/60D21B6E/60F5ADAC/614E5539" Ref="C43"  Part="1"
-F 0 "C43" H 6465 3446 50  0000 L CNN
+F 0 "C44" H 6465 3446 50  0000 L CNN
 F 1 "10u" H 6465 3355 50  0000 L CNN
-F 2 "Capacitor_SMD:C_0402_1005Metric" H 6388 3250 50  0001 C CNN
+F 2 "Capacitor_SMD:C_0603_1608Metric_Pad1.08x0.95mm_HandSolder" H 6388 3250 50  0001 C CNN
 F 3 "~" H 6350 3400 50  0001 C CNN
 	1    6350 3400
@@
 AR Path="/60D21B6E/6160D475/614E55C8" Ref="R15"  Part="1"
 AR Path="/60D21B6E/60F5ADAC/614E55C8" Ref="R24"  Part="1"
-F 0 "R24" V 5650 3650 50  0000 C CNN
+F 0 "R12" V 5650 3650 50  0000 C CNN
 F 1 "174" V 5750 3650 50  0000 C CNN
-F 2 "Resistor_SMD:R_0402_1005Metric" V 5680 3650 50  0001 C CNN
+F 2 "Resistor_SMD:R_0603_1608Metric_Pad0.98x0.95mm_HandSolder" V 5680 3650 50  0001 C CNN
 F 3 "~" H 5750 3650 50  0001 C CNN
 	1    5750 3650
@@
 AR Path="/60D21B6E/6160D475/614E5545" Ref="TR2"  Part="1"
 AR Path="/60D21B6E/60F5ADAC/614E5545" Ref="TR2"  Part="1"
-F 0 "TR2" H 7150 3581 50  0000 C CNN
+F 0 "TR1" H 7150 3581 50  0000 C CNN
 F 1 "ADT2-1T" H 7150 3490 50  0000 C CNN
 F 2 "RF_Mini-Circuits:Mini-Circuits_CD542_H2.84mm" H 7150 2850 50  0001 C CNN

Commit message: Added options for the tranfo
Parts:
- added R18, R20: 0, Resistor_SMD:R_0603_1608Metric_Pad0.98x0.95mm_HandSolder, symbol Device:R
Connections:
- net CMO: now also R18.2
- net GND: now also R20.2; no longer TR1.1
- new net: R18.1, R20.1, TR1.1
Changed lines of the file:
@@
 AR Path="/60D21B6E/6160D475/614E557C" Ref="#PWR0140"  Part="1"
 AR Path="/60D21B6E/60F5ADAC/614E557C" Ref="#PWR0139"  Part="1"
-F 0 "#PWR0139" H 6350 3400 50  0001 C CNN
+F 0 "#PWR0128" H 6350 3400 50  0001 C CNN
 F 1 "GND" H 6355 3477 50  0000 C CNN
 F 2 "" H 6350 3650 50  0001 C CNN
@@
 L power:GND #PWR?
 U 1 1 614E5583
-P 7500 3450
+P 7500 3800
 AR Path="/60D21B6E/614E5583" Ref="#PWR?"  Part="1"
 AR Path="/60D21B6E/60D8B1A1/614E5583" Ref="#PWR0130"  Part="1"
@@
 AR Path="/60D21B6E/6160D475/614E5583" Ref="#PWR0142"  Part="1"
 AR Path="/60D21B6E/60F5ADAC/614E5583" Ref="#PWR0140"  Part="1"
-F 0 "#PWR0140" H 7500 3200 50  0001 C CNN
-F 1 "GND" H 7505 3277 50  0000 C CNN
-F 2 "" H 7500 3450 50  0001 C CNN
-F 3 "" H 7500 3450 50  0001 C CNN
-	1    7500 3450
+F 0 "#PWR0130" H 7500 3550 50  0001 C CNN
+F 1 "GND" H 7505 3627 50  0000 C CNN
+F 2 "" H 7500 3800 50  0001 C CNN
+F 3 "" H 7500 3800 50  0001 C CNN
+	1    7500 3800
 	-1   0    0    -1
 $EndComp
@@
 Wire Wire Line
 	6850 3400 6950 3400
-Wire Wire Line
-	7350 3400 7500 3400
 Wire Wire Line
 	7500 3400 7500 3450
@@
 Wire Wire Line
 	7350 3000 8050 3000
+$Comp
+L Device:R R?
+U 1 1 6147DECF
+P 7700 3400
+AR Path="/60D21B6E/6147DECF" Ref="R?"  Part="1"
+AR Path="/60D21B6E/60D894BC/6147DECF" Ref="R?"  Part="1"
+AR Path="/60D21B6E/6110419F/6147DECF" Ref="R?"  Part="1"
+AR Path="/60D21B6E/61121120/6147DECF" Ref="R?"  Part="1"
+AR Path="/60D21B6E/60F52DEE/6147DECF" Ref="R?"  Part="1"
+AR Path="/60D21B6E/60D8B1A1/6147DECF" Ref="R18"  Part="1"
+AR Path="/60D21B6E/60F5ADAC/6147DECF" Ref="R40"  Part="1"
+F 0 "R18" H 7770 3446 50  0000 L CNN
+F 1 "0" V 7700 3350 50  0000 L CNN
+F 2 "Resistor_SMD:R_0603_1608Metric_Pad0.98x0.95mm_HandSolder" V 7630 3400 50  0001 C CNN
+F 3 "~" H 7700 3400 50  0001 C CNN
+	1    7700 3400
+	0    -1   -1   0
+$EndComp
+$Comp
+L Device:R R?
+U 1 1 6147DED5
+P 7500 3600
+AR Path="/60D21B6E/6147DED5" Ref="R?"  Part="1"
+AR Path="/60D21B6E/60D894BC/6147DED5" Ref="R?"  Part="1"
+AR Path="/60D21B6E/6110419F/6147DED5" Ref="R?"  Part="1"
+AR Path="/60D21B6E/61121120/6147DED5" Ref="R?"  Part="1"
+AR Path="/60D21B6E/60F52DEE/6147DED5" Ref="R?"  Part="1"
+AR Path="/60D21B6E/60D8B1A1/6147DED5" Ref="R20"  Part="1"
+AR Path="/60D21B6E/60F5ADAC/6147DED5" Ref="R41"  Part="1"
+F 0 "R20" H 7570 3646 50  0000 L CNN
+F 1 "0" V 7500 3550 50  0000 L CNN
+F 2 "Resistor_SMD:R_0603_1608Metric_Pad0.98x0.95mm_HandSolder" V 7430 3600 50  0001 C CNN
+F 3 "~" H 7500 3600 50  0001 C CNN
+	1    7500 3600
+	1    0    0    -1
+$EndComp
+Wire Wire Line
+	7500 3400 7550 3400
+Wire Wire Line
+	7500 3750 7500 3800
+Text GLabel 7950 3400 2    50   Input ~ 0
+CMO
+Wire Wire Line
+	7950 3400 7850 3400
+Wire Wire Line
+	7350 3400 7500 3400
+Connection ~ 7500 3400
 $EndSCHEMATC

Commit message: added the option to switch HMC860 for HMC1060
Changed lines of the file:
@@
 AR Path="/60D21B6E/6160D475/614E552D" Ref="R16"  Part="1"
 AR Path="/60D21B6E/60F5ADAC/614E552D" Ref="R16"  Part="1"
-F 0 "R11" H 5980 3254 50  0000 R CNN
+F 0 "R16" H 5980 3254 50  0000 R CNN
 F 1 "140" H 5980 3345 50  0000 R CNN
 F 2 "Resistor_SMD:R_0603_1608Metric_Pad0.98x0.95mm_HandSolder" V 5980 3300 50  0001 C CNN
@@
 AR Path="/60D21B6E/6160D475/614E5533" Ref="R24"  Part="1"
 AR Path="/60D21B6E/60F5ADAC/614E5533" Ref="R15"  Part="1"
-F 0 "R21" V 5650 2950 50  0000 C CNN
+F 0 "R15" V 5650 2950 50  0000 C CNN
 F 1 "174" V 5750 2950 50  0000 C CNN
 F 2 "Resistor_SMD:R_0603_1608Metric_Pad0.98x0.95mm_HandSolder" V 5680 2950 50  0001 C CNN
@@
 AR Path="/60D21B6E/6160D475/614E5539" Ref="C43"  Part="1"
 AR Path="/60D21B6E/60F5ADAC/614E5539" Ref="C43"  Part="1"
-F 0 "C44" H 6465 3446 50  0000 L CNN
+F 0 "C43" H 6465 3446 50  0000 L CNN
 F 1 "10u" H 6465 3355 50  0000 L CNN
 F 2 "Capacitor_SMD:C_0603_1608Metric_Pad1.08x0.95mm_HandSolder" H 6388 3250 50  0001 C CNN
@@
 AR Path="/60D21B6E/6160D475/614E557C" Ref="#PWR0140"  Part="1"
 AR Path="/60D21B6E/60F5ADAC/614E557C" Ref="#PWR0139"  Part="1"
-F 0 "#PWR0128" H 6350 3400 50  0001 C CNN
+F 0 "#PWR0139" H 6350 3400 50  0001 C CNN
 F 1 "GND" H 6355 3477 50  0000 C CNN
 F 2 "" H 6350 3650 50  0001 C CNN
@@
 AR Path="/60D21B6E/6160D475/614E55C8" Ref="R15"  Part="1"
 AR Path="/60D21B6E/60F5ADAC/614E55C8" Ref="R24"  Part="1"
-F 0 "R12" V 5650 3650 50  0000 C CNN
+F 0 "R24" V 5650 3650 50  0000 C CNN
 F 1 "174" V 5750 3650 50  0000 C CNN
 F 2 "Resistor_SMD:R_0603_1608Metric_Pad0.98x0.95mm_HandSolder" V 5680 3650 50  0001 C CNN
@@
 AR Path="/60D21B6E/6160D475/614E5583" Ref="#PWR0142"  Part="1"
 AR Path="/60D21B6E/60F5ADAC/614E5583" Ref="#PWR0140"  Part="1"
-F 0 "#PWR0130" H 7500 3550 50  0001 C CNN
+F 0 "#PWR0140" H 7500 3550 50  0001 C CNN
 F 1 "GND" H 7505 3627 50  0000 C CNN
 F 2 "" H 7500 3800 50  0001 C CNN
@@
 AR Path="/60D21B6E/60F5ADAC/614E5545" Ref="TR2"  Part="1"
 AR Path="/614E5545" Ref="TR1"  Part="1"
-F 0 "TR1" H 7150 3581 50  0000 C CNN
+F 0 "TR2" H 7150 3581 50  0000 C CNN
 F 1 "ADT2-1T" H 7150 3490 50  0000 C CNN
 F 2 "RF_Mini-Circuits:Mini-Circuits_CD542_H2.84mm" H 7150 2850 50  0001 C CNN
@@
 AR Path="/60D21B6E/60D8B1A1/6147DECF" Ref="R18"  Part="1"
 AR Path="/60D21B6E/60F5ADAC/6147DECF" Ref="R40"  Part="1"
-F 0 "R18" H 7770 3446 50  0000 L CNN
+F 0 "R40" H 7770 3446 50  0000 L CNN
 F 1 "0" V 7700 3350 50  0000 L CNN
 F 2 "Resistor_SMD:R_0603_1608Metric_Pad0.98x0.95mm_HandSolder" V 7630 3400 50  0001 C CNN
@@
 AR Path="/60D21B6E/60D8B1A1/6147DED5" Ref="R20"  Part="1"
 AR Path="/60D21B6E/60F5ADAC/6147DED5" Ref="R41"  Part="1"
-F 0 "R20" H 7570 3646 50  0000 L CNN
+F 0 "R41" H 7570 3646 50  0000 L CNN
 F 1 "0" V 7500 3550 50  0000 L CNN
 F 2 "Resistor_SMD:R_0603_1608Metric_Pad0.98x0.95mm_HandSolder" V 7430 3600 50  0001 C CNN

Commit message: As implemented for v1
Parts:
- R18: value 0 -> 0(NP)
Changed lines of the file:
@@
 AR Path="/60D21B6E/6160D475/614E552D" Ref="R16"  Part="1"
 AR Path="/60D21B6E/60F5ADAC/614E552D" Ref="R16"  Part="1"
-F 0 "R16" H 5980 3254 50  0000 R CNN
+F 0 "R11" H 5980 3254 50  0000 R CNN
 F 1 "140" H 5980 3345 50  0000 R CNN
 F 2 "Resistor_SMD:R_0603_1608Metric_Pad0.98x0.95mm_HandSolder" V 5980 3300 50  0001 C CNN
@@
 AR Path="/60D21B6E/6160D475/614E5533" Ref="R24"  Part="1"
 AR Path="/60D21B6E/60F5ADAC/614E5533" Ref="R15"  Part="1"
-F 0 "R15" V 5650 2950 50  0000 C CNN
+F 0 "R21" V 5650 2950 50  0000 C CNN
 F 1 "174" V 5750 2950 50  0000 C CNN
 F 2 "Resistor_SMD:R_0603_1608Metric_Pad0.98x0.95mm_HandSolder" V 5680 2950 50  0001 C CNN
@@
 AR Path="/60D21B6E/6160D475/614E5539" Ref="C43"  Part="1"
 AR Path="/60D21B6E/60F5ADAC/614E5539" Ref="C43"  Part="1"
-F 0 "C43" H 6465 3446 50  0000 L CNN
+F 0 "C44" H 6465 3446 50  0000 L CNN
 F 1 "10u" H 6465 3355 50  0000 L CNN
 F 2 "Capacitor_SMD:C_0603_1608Metric_Pad1.08x0.95mm_HandSolder" H 6388 3250 50  0001 C CNN
@@
 AR Path="/60D21B6E/6160D475/614E557C" Ref="#PWR0140"  Part="1"
 AR Path="/60D21B6E/60F5ADAC/614E557C" Ref="#PWR0139"  Part="1"
-F 0 "#PWR0139" H 6350 3400 50  0001 C CNN
+F 0 "#PWR0128" H 6350 3400 50  0001 C CNN
 F 1 "GND" H 6355 3477 50  0000 C CNN
 F 2 "" H 6350 3650 50  0001 C CNN
@@
 AR Path="/60D21B6E/6160D475/614E55C8" Ref="R15"  Part="1"
 AR Path="/60D21B6E/60F5ADAC/614E55C8" Ref="R24"  Part="1"
-F 0 "R24" V 5650 3650 50  0000 C CNN
+F 0 "R12" V 5650 3650 50  0000 C CNN
 F 1 "174" V 5750 3650 50  0000 C CNN
 F 2 "Resistor_SMD:R_0603_1608Metric_Pad0.98x0.95mm_HandSolder" V 5680 3650 50  0001 C CNN
@@
 AR Path="/60D21B6E/6160D475/614E5583" Ref="#PWR0142"  Part="1"
 AR Path="/60D21B6E/60F5ADAC/614E5583" Ref="#PWR0140"  Part="1"
-F 0 "#PWR0140" H 7500 3550 50  0001 C CNN
+F 0 "#PWR0130" H 7500 3550 50  0001 C CNN
 F 1 "GND" H 7505 3627 50  0000 C CNN
 F 2 "" H 7500 3800 50  0001 C CNN
@@
 AR Path="/60D21B6E/60F5ADAC/614E5545" Ref="TR2"  Part="1"
 AR Path="/614E5545" Ref="TR1"  Part="1"
-F 0 "TR2" H 7150 3581 50  0000 C CNN
+F 0 "TR1" H 7150 3581 50  0000 C CNN
 F 1 "ADT2-1T" H 7150 3490 50  0000 C CNN
 F 2 "RF_Mini-Circuits:Mini-Circuits_CD542_H2.84mm" H 7150 2850 50  0001 C CNN
@@
 AR Path="/60D21B6E/60D8B1A1/6147DECF" Ref="R18"  Part="1"
 AR Path="/60D21B6E/60F5ADAC/6147DECF" Ref="R40"  Part="1"
-F 0 "R40" H 7770 3446 50  0000 L CNN
-F 1 "0" V 7700 3350 50  0000 L CNN
+F 0 "R18" H 7770 3446 50  0000 L CNN
+F 1 "0(NP)" V 7700 3275 50  0000 L CNN
 F 2 "Resistor_SMD:R_0603_1608Metric_Pad0.98x0.95mm_HandSolder" V 7630 3400 50  0001 C CNN
 F 3 "~" H 7700 3400 50  0001 C CNN
@@
 AR Path="/60D21B6E/60D8B1A1/6147DED5" Ref="R20"  Part="1"
 AR Path="/60D21B6E/60F5ADAC/6147DED5" Ref="R41"  Part="1"
-F 0 "R41" H 7570 3646 50  0000 L CNN
+F 0 "R20" H 7570 3646 50  0000 L CNN
 F 1 "0" V 7500 3550 50  0000 L CNN
 F 2 "Resistor_SMD:R_0603_1608Metric_Pad0.98x0.95mm_HandSolder" V 7430 3600 50  0001 C CNN

Commit message: removed unused options added aop at the output
Parts:
- removed R18: 0(NP), Resistor_SMD:R_0603_1608Metric_Pad0.98x0.95mm_HandSolder, symbol Device:R
- removed R20: 0, Resistor_SMD:R_0603_1608Metric_Pad0.98x0.95mm_HandSolder, symbol Device:R
Connections:
- net CMI: now reaches TR1.1
Changed lines of the file:
@@
 AR Path="/60D21B6E/6160D475/614E552D" Ref="R16"  Part="1"
 AR Path="/60D21B6E/60F5ADAC/614E552D" Ref="R16"  Part="1"
-F 0 "R11" H 5980 3254 50  0000 R CNN
+F 0 "R16" H 5980 3254 50  0000 R CNN
 F 1 "140" H 5980 3345 50  0000 R CNN
 F 2 "Resistor_SMD:R_0603_1608Metric_Pad0.98x0.95mm_HandSolder" V 5980 3300 50  0001 C CNN
@@
 AR Path="/60D21B6E/6160D475/614E5533" Ref="R24"  Part="1"
 AR Path="/60D21B6E/60F5ADAC/614E5533" Ref="R15"  Part="1"
-F 0 "R21" V 5650 2950 50  0000 C CNN
+F 0 "R15" V 5650 2950 50  0000 C CNN
 F 1 "174" V 5750 2950 50  0000 C CNN
 F 2 "Resistor_SMD:R_0603_1608Metric_Pad0.98x0.95mm_HandSolder" V 5680 2950 50  0001 C CNN
@@
 AR Path="/60D21B6E/6160D475/614E5539" Ref="C43"  Part="1"
 AR Path="/60D21B6E/60F5ADAC/614E5539" Ref="C43"  Part="1"
-F 0 "C44" H 6465 3446 50  0000 L CNN
+F 0 "C43" H 6465 3446 50  0000 L CNN
 F 1 "10u" H 6465 3355 50  0000 L CNN
 F 2 "Capacitor_SMD:C_0603_1608Metric_Pad1.08x0.95mm_HandSolder" H 6388 3250 50  0001 C CNN
@@
 AR Path="/60D21B6E/6160D475/614E557C" Ref="#PWR0140"  Part="1"
 AR Path="/60D21B6E/60F5ADAC/614E557C" Ref="#PWR0139"  Part="1"
-F 0 "#PWR0128" H 6350 3400 50  0001 C CNN
+F 0 "#PWR0139" H 6350 3400 50  0001 C CNN
 F 1 "GND" H 6355 3477 50  0000 C CNN
 F 2 "" H 6350 3650 50  0001 C CNN
@@
 AR Path="/60D21B6E/6160D475/614E55C8" Ref="R15"  Part="1"
 AR Path="/60D21B6E/60F5ADAC/614E55C8" Ref="R24"  Part="1"
-F 0 "R12" V 5650 3650 50  0000 C CNN
+F 0 "R24" V 5650 3650 50  0000 C CNN
 F 1 "174" V 5750 3650 50  0000 C CNN
 F 2 "Resistor_SMD:R_0603_1608Metric_Pad0.98x0.95mm_HandSolder" V 5680 3650 50  0001 C CNN
@@
 Wire Wire Line
 	6350 3550 6350 3650
-$Comp
-L power:GND #PWR?
-U 1 1 614E5583
-P 7500 3800
-AR Path="/60D21B6E/614E5583" Ref="#PWR?"  Part="1"
-AR Path="/60D21B6E/60D8B1A1/614E5583" Ref="#PWR0130"  Part="1"
-AR Path="/60D21B6E/6152EBAF/614E5583" Ref="#PWR?"  Part="1"
-AR Path="/60D21B6E/615DF219/614E5583" Ref="#PWR?"  Part="1"
-AR Path="/60D21B6E/615DFEB1/614E5583" Ref="#PWR?"  Part="1"
-AR Path="/60D21B6E/615E1BD1/614E5583" Ref="#PWR?"  Part="1"
-AR Path="/60D21B6E/6160D475/614E5583" Ref="#PWR0142"  Part="1"
-AR Path="/60D21B6E/60F5ADAC/614E5583" Ref="#PWR0140"  Part="1"
-F 0 "#PWR0130" H 7500 3550 50  0001 C CNN
-F 1 "GND" H 7505 3627 50  0000 C CNN
-F 2 "" H 7500 3800 50  0001 C CNN
-F 3 "" H 7500 3800 50  0001 C CNN
-	1    7500 3800
-	-1   0    0    -1
-$EndComp
 Wire Wire Line
 	6850 3000 6950 3000
@@
 Wire Wire Line
 	6850 3400 6950 3400
-Wire Wire Line
-	7500 3400 7500 3450
 $Comp
 L LibPersoNadj:ADT2-1T TR?
@@
 AR Path="/60D21B6E/60F5ADAC/614E5545" Ref="TR2"  Part="1"
 AR Path="/614E5545" Ref="TR1"  Part="1"
-F 0 "TR1" H 7150 3581 50  0000 C CNN
+F 0 "TR2" H 7150 3581 50  0000 C CNN
 F 1 "ADT2-1T" H 7150 3490 50  0000 C CNN
 F 2 "RF_Mini-Circuits:Mini-Circuits_CD542_H2.84mm" H 7150 2850 50  0001 C CNN
@@
 Wire Wire Line
 	7350 3000 8050 3000
-$Comp
-L Device:R R?
-U 1 1 6147DECF
-P 7700 3400
-AR Path="/60D21B6E/6147DECF" Ref="R?"  Part="1"
-AR Path="/60D21B6E/60D894BC/6147DECF" Ref="R?"  Part="1"
-AR Path="/60D21B6E/6110419F/6147DECF" Ref="R?"  Part="1"
-AR Path="/60D21B6E/61121120/6147DECF" Ref="R?"  Part="1"
-AR Path="/60D21B6E/60F52DEE/6147DECF" Ref="R?"  Part="1"
-AR Path="/60D21B6E/60D8B1A1/6147DECF" Ref="R18"  Part="1"
-AR Path="/60D21B6E/60F5ADAC/6147DECF" Ref="R40"  Part="1"
-F 0 "R18" H 7770 3446 50  0000 L CNN
-F 1 "0(NP)" V 7700 3275 50  0000 L CNN
-F 2 "Resistor_SMD:R_0603_1608Metric_Pad0.98x0.95mm_HandSolder" V 7630 3400 50  0001 C CNN
-F 3 "~" H 7700 3400 50  0001 C CNN
-	1    7700 3400
-	0    -1   -1   0
-$EndComp
-$Comp
-L Device:R R?
-U 1 1 6147DED5
-P 7500 3600
-AR Path="/60D21B6E/6147DED5" Ref="R?"  Part="1"
-AR Path="/60D21B6E/60D894BC/6147DED5" Ref="R?"  Part="1"
-AR Path="/60D21B6E/6110419F/6147DED5" Ref="R?"  Part="1"
-AR Path="/60D21B6E/61121120/6147DED5" Ref="R?"  Part="1"
-AR Path="/60D21B6E/60F52DEE/6147DED5" Ref="R?"  Part="1"
-AR Path="/60D21B6E/60D8B1A1/6147DED5" Ref="R20"  Part="1"
-AR Path="/60D21B6E/60F5ADAC/6147DED5" Ref="R41"  Part="1"
-F 0 "R20" H 7570 3646 50  0000 L CNN
-F 1 "0" V 7500 3550 50  0000 L CNN
-F 2 "Resistor_SMD:R_0603_1608Metric_Pad0.98x0.95mm_HandSolder" V 7430 3600 50  0001 C CNN
-F 3 "~" H 7500 3600 50  0001 C CNN
-	1    7500 3600
-	1    0    0    -1
-$EndComp
 Wire Wire Line
-	7500 3400 7550 3400
-Wire Wire Line
-	7500 3750 7500 3800
-Text GLabel 7950 3400 2    50   Input ~ 0
-CMO
-Wire Wire Line
-	7950 3400 7850 3400
-Wire Wire Line
-	7350 3400 7500 3400
-Connection ~ 7500 3400
+	7350 3400 7450 3400
+Text GLabel 7450 3400 2    50   Input ~ 0
+CMI
 $EndSCHEMATC

Commit message: output tranfo and aop work around vdd/2 caped aop's amplification at 9dB
Changed lines of the file:
@@
 AR Path="/60D21B6E/6160D475/614E552D" Ref="R16"  Part="1"
 AR Path="/60D21B6E/60F5ADAC/614E552D" Ref="R16"  Part="1"
-F 0 "R16" H 5980 3254 50  0000 R CNN
+F 0 "R11" H 5980 3254 50  0000 R CNN
 F 1 "140" H 5980 3345 50  0000 R CNN
 F 2 "Resistor_SMD:R_0603_1608Metric_Pad0.98x0.95mm_HandSolder" V 5980 3300 50  0001 C CNN
@@
 AR Path="/60D21B6E/6160D475/614E5533" Ref="R24"  Part="1"
 AR Path="/60D21B6E/60F5ADAC/614E5533" Ref="R15"  Part="1"
-F 0 "R15" V 5650 2950 50  0000 C CNN
+F 0 "R21" V 5650 2950 50  0000 C CNN
 F 1 "174" V 5750 2950 50  0000 C CNN
 F 2 "Resistor_SMD:R_0603_1608Metric_Pad0.98x0.95mm_HandSolder" V 5680 2950 50  0001 C CNN
@@
 AR Path="/60D21B6E/6160D475/614E5539" Ref="C43"  Part="1"
 AR Path="/60D21B6E/60F5ADAC/614E5539" Ref="C43"  Part="1"
-F 0 "C43" H 6465 3446 50  0000 L CNN
+F 0 "C44" H 6465 3446 50  0000 L CNN
 F 1 "10u" H 6465 3355 50  0000 L CNN
 F 2 "Capacitor_SMD:C_0603_1608Metric_Pad1.08x0.95mm_HandSolder" H 6388 3250 50  0001 C CNN
@@
 AR Path="/60D21B6E/6160D475/614E557C" Ref="#PWR0140"  Part="1"
 AR Path="/60D21B6E/60F5ADAC/614E557C" Ref="#PWR0139"  Part="1"
-F 0 "#PWR0139" H 6350 3400 50  0001 C CNN
+F 0 "#PWR0128" H 6350 3400 50  0001 C CNN
 F 1 "GND" H 6355 3477 50  0000 C CNN
 F 2 "" H 6350 3650 50  0001 C CNN
@@
 AR Path="/60D21B6E/6160D475/614E55C8" Ref="R15"  Part="1"
 AR Path="/60D21B6E/60F5ADAC/614E55C8" Ref="R24"  Part="1"
-F 0 "R24" V 5650 3650 50  0000 C CNN
+F 0 "R12" V 5650 3650 50  0000 C CNN
 F 1 "174" V 5750 3650 50  0000 C CNN
 F 2 "Resistor_SMD:R_0603_1608Metric_Pad0.98x0.95mm_HandSolder" V 5680 3650 50  0001 C CNN
@@
 AR Path="/60D21B6E/60F5ADAC/614E5545" Ref="TR2"  Part="1"
 AR Path="/614E5545" Ref="TR1"  Part="1"
-F 0 "TR2" H 7150 3581 50  0000 C CNN
+F 0 "TR1" H 7150 3581 50  0000 C CNN
 F 1 "ADT2-1T" H 7150 3490 50  0000 C CNN
 F 2 "RF_Mini-Circuits:Mini-Circuits_CD542_H2.84mm" H 7150 2850 50  0001 C CNN
