File: Bifrost.sch (KiCad schematic (older format))
At the start: 18 parts, among them J1 OIP, J10 SSW-106-01-T-D, J4 OQP, J5 CalCK

Commit message: Corrected errors from single ended transition
Parts:
- removed J10: SSW-106-01-T-D, Connector_PinHeader_2.54mm:PinHeader_2x06_P2.54mm_Vertical, symbol Connector_Generic:Conn_02x06_Odd_Even
- removed R48, R51, R54, R55: DEPOP, Resistor_SMD:R_0402_1005Metric, symbol Device:R
- added AD1: Conn_01x06_Female, Connector_PinHeader_2.54mm:PinHeader_1x06_P2.54mm_Vertical, symbol Connector:Conn_01x06_Female
- added H1, H2, H3, H4: MountingHole, MountingHole:MountingHole_3mm, symbol Mechanical:MountingHole
- added ICSP1, ICSP2: Conn_02x03_Odd_Even, Connector_PinSocket_2.54mm:PinSocket_2x03_P2.54mm_Vertical, symbol Connector_Generic:Conn_02x03_Odd_Even
- added IOH1: Conn_01x10_Female, Connector_PinHeader_2.54mm:PinHeader_1x10_P2.54mm_Vertical, symbol Connector:Conn_01x10_Female
- added IOL1, POWER1: Conn_01x08_Female, Connector_PinHeader_2.54mm:PinHeader_1x08_P2.54mm_Vertical, symbol Connector:Conn_01x08_Female
- gave numbers to parts that had none: 4
Connections:
- net labels added: +3V3, +5V, AD0, AD1, AD2, AD3, AD4, AD4/SDA, AD5, AD5/SCL, AREF, IO0, IO1, IO2, IO3, IO4, IO5, IO6, IO7, IO8, IO9, MISO, MISO2, MOSI, MOSI2, RESET, RESET2, SCK2, SCK_S, SDI_S, SDO_S, SEN_S, SS, VIN
- wire segments 71 -> 99
- no-connect marks 5 -> 1
Other:
- note added: "0"
- note added: "1"
- note added: "10"
- note added: "11"
- note added: "12"
- note added: "13"
- note added: "2"
- note added: "3"
- note added: "4"
- note added: "5"
- note added: "6"
- note added: "7"
- note added: "8"
- note added: "9"
- note added: "SCL"
- note added: "SDA"
- moved on the sheet: IC1, IC2, J1, J4, J5, R49, R52, R53, R56, R71, R72

Commit message: passage 0402 => 0603
Parts:
- removed TP2: +5.5V, TestPoint:TestPoint_Loop_D2.60mm_Drill1.6mm_Beaded, symbol Connector:TestPoint
- removed TP3: GND, TestPoint:TestPoint_Loop_D2.60mm_Drill1.6mm_Beaded, symbol Connector:TestPoint
- added J?: Barrel_Jack_Switch, symbol Connector:Barrel_Jack_Switch
- added R100: 0, Resistor_SMD:R_0603_1608Metric_Pad0.98x0.95mm_HandSolder, symbol Device:R
- R49, R52, R53, R56, R71, R72: footprint Resistor_SMD:R_0402_1005Metric -> Resistor_SMD:R_0603_1608Metric_Pad0.98x0.95mm_HandSolder
Connections:
- net labels added: +5V_Ard
- net labels removed: AD4/SDA, AD5/SCL
- wire segments 99 -> 106
- no-connect marks 1 -> 21
Changed lines of the file:
@@
 	7650 1600 7650 1650
 $Sheet
-S 1400 2950 900  350
+S 1600 3100 900  350
 U 6188E6DD
 F0 "Sheet6188E6DC" 50
 F1 "AlimHMC860.sch" 50
-F2 "5.5V" I L 1400 3100 50
+F2 "5.5V" I L 1600 3250 50
 $EndSheet
 Wire Wire Line
-	1400 3100 1150 3100
-Wire Wire Line
-	1150 3600 900  3600
+	1600 3250 1350 3250
+Wire Wire Line
+	1350 3750 1100 3750
 $Comp
 L power:GND #PWR?
 U 1 1 61AEA5FE
-P 1150 3850
+P 1350 4000
 AR Path="/60D21B6E/61AEA5FE" Ref="#PWR?"  Part="1"
 AR Path="/61AEA5FE" Ref="#PWR0156"  Part="1"
-F 0 "#PWR0156" H 1150 3600 50  0001 C CNN
-F 1 "GND" H 1155 3677 50  0000 C CNN
-F 2 "" H 1150 3850 50  0001 C CNN
-F 3 "" H 1150 3850 50  0001 C CNN
-	1    1150 3850
-	1    0    0    -1
-$EndComp
-Wire Wire Line
-	1150 3600 1150 3850
-$Comp
-L Connector:TestPoint TP2
-U 1 1 61B13AF5
-P 900 3100
-F 0 "TP2" V 1095 3172 50  0000 C CNN
-F 1 "+5.5V" V 1004 3172 50  0000 C CNN
-F 2 "TestPoint:TestPoint_Loop_D2.60mm_Drill1.6mm_Beaded" H 1100 3100 50  0001 C CNN
-F 3 "~" H 1100 3100 50  0001 C CNN
-	1    900  3100
-	0    -1   -1   0
-$EndComp
-$Comp
-L Connector:TestPoint TP3
-U 1 1 61B14AC1
-P 900 3600
-F 0 "TP3" V 1095 3672 50  0000 C CNN
-F 1 "GND" V 1004 3672 50  0000 C CNN
-F 2 "TestPoint:TestPoint_Loop_D2.60mm_Drill1.6mm_Beaded" H 1100 3600 50  0001 C CNN
-F 3 "~" H 1100 3600 50  0001 C CNN
-	1    900  3600
-	0    -1   -1   0
-$EndComp
+F 0 "#PWR0156" H 1350 3750 50  0001 C CNN
+F 1 "GND" H 1355 3827 50  0000 C CNN
+F 2 "" H 1350 4000 50  0001 C CNN
+F 3 "" H 1350 4000 50  0001 C CNN
+	1    1350 4000
+	1    0    0    -1
+$EndComp
+Wire Wire Line
+	1350 3750 1350 4000
 $Comp
 L power:PWR_FLAG #FLG0107
 U 1 1 61B17BC7
-P 1150 3000
-F 0 "#FLG0107" H 1150 3075 50  0001 C CNN
-F 1 "PWR_FLAG" H 1150 3173 50  0000 C CNN
-F 2 "" H 1150 3000 50  0001 C CNN
-F 3 "~" H 1150 3000 50  0001 C CNN
-	1    1150 3000
-	1    0    0    -1
-$EndComp
-$Comp
-L power:PWR_FLAG #FLG0108
-U 1 1 61B189E4
-P 1150 3500
-F 0 "#FLG0108" H 1150 3575 50  0001 C CNN
-F 1 "PWR_FLAG" H 1150 3673 50  0000 C CNN
-F 2 "" H 1150 3500 50  0001 C CNN
-F 3 "~" H 1150 3500 50  0001 C CNN
-	1    1150 3500
-	1    0    0    -1
-$EndComp
-Wire Wire Line
-	1150 3000 1150 3100
-Connection ~ 1150 3100
-Wire Wire Line
-	1150 3100 900  3100
-Wire Wire Line
-	1150 3500 1150 3600
-Connection ~ 1150 3600
+P 1350 3150
+F 0 "#FLG0107" H 1350 3225 50  0001 C CNN
+F 1 "PWR_FLAG" H 1350 3323 50  0000 C CNN
+F 2 "" H 1350 3150 50  0001 C CNN
+F 3 "~" H 1350 3150 50  0001 C CNN
+	1    1350 3150
+	1    0    0    -1
+$EndComp
+Wire Wire Line
+	1350 3150 1350 3250
+Connection ~ 1350 3250
+Wire Wire Line
+	1350 3250 1100 3250
+Wire Wire Line
+	1350 3650 1350 3750
+Connection ~ 1350 3750
 $Comp
 L LibPersoNadj:DS1085Z-10+ IC1
@@
 F 0 "R71" V 4850 1200 50  0000 C CNN
 F 1 "510" V 4900 1000 50  0000 C CNN
-F 2 "Resistor_SMD:R_0402_1005Metric" V 4830 1000 50  0001 C CNN
+F 2 "Resistor_SMD:R_0603_1608Metric_Pad0.98x0.95mm_HandSolder" V 4830 1000 50  0001 C CNN
 F 3 "~" H 4900 1000 50  0001 C CNN
 	1    4900 1000
@@
 F 0 "R72" V 4850 2150 50  0000 C CNN
 F 1 "510" V 4900 1950 50  0000 C CNN
-F 2 "Resistor_SMD:R_0402_1005Metric" V 4830 1950 50  0001 C CNN
+F 2 "Resistor_SMD:R_0603_1608Metric_Pad0.98x0.95mm_HandSolder" V 4830 1950 50  0001 C CNN
 F 3 "~" H 4900 1950 50  0001 C CNN
 	1    4900 1950
@@
 AD4
 Text Label 9950 2850 0    70   ~ 0
-AD4/SDA
+SDA
 Text Label 800  5500 0    70   ~ 0
 AD5
 Text Label 9950 2750 0    70   ~ 0
-AD5/SCL
+SCL
 Text Label 10250 6000 0    70   ~ 0
 IO2
@@
 	1    0    0    -1
 $EndComp
-Text Label 850  1100 0    70   ~ 0
+Text Label 650  1100 0    70   ~ 0
 +3V3
 Wire Wire Line
-	1600 1100 800  1100
-Text Label 1000 1500 0    70   ~ 0
-VIN
-Wire Wire Line
-	1000 1500 1600 1500
-Wire Wire Line
-	1600 1400 800  1400
-Wire Wire Line
-	1600 1300 800  1300
-Wire Wire Line
-	800  1300 800  1400
-Text Label 800  1200 0    10   ~ 0
-+5V
+	1600 1100 600  1100
+Wire Wire Line
+	1600 1400 600  1400
+Wire Wire Line
+	1600 1300 600  1300
+Wire Wire Line
+	600  1300 600  1400
 Text Notes 10825 3500 0    59   ~ 0
 10
-Text Label 800  1300 0    10   ~ 0
+Text Label 600  1300 0    10   ~ 0
 GND
 Text Label 10500 1400 0    10   ~ 0
 GND
-Connection ~ 800  1400
-Wire Wire Line
-	800  1400 800  1500
+Connection ~ 600  1400
+Wire Wire Line
+	600  1400 600  1500
 Wire Wire Line
 	10500 1400 10700 1400
@@
 	1    0    0    -1
 $EndComp
-Text Label 800  1000 0    66   ~ 0
+Text Label 600  1000 0    66   ~ 0
 RESET
 Text Label 7700 600  0    10   ~ 0
 GND
 Wire Wire Line
-	1300 1200 800  1200
+	1300 1200 600  1200
 Wire Wire Line
 	1600 1200 1300 1200
@@
 L power:GND #PWR0101
 U 1 1 614371B4
-P 800 1500
-F 0 "#PWR0101" H 800 1250 50  0001 C CNN
-F 1 "GND" H 805 1327 50  0000 C CNN
-F 2 "" H 800 1500 50  0001 C CNN
-F 3 "" H 800 1500 50  0001 C CNN
-	1    800  1500
+P 600 1500
+F 0 "#PWR0101" H 600 1250 50  0001 C CNN
+F 1 "GND" H 605 1327 50  0000 C CNN
+F 2 "" H 600 1500 50  0001 C CNN
+F 3 "" H 600 1500 50  0001 C CNN
+	1    600  1500
 	1    0    0    -1
 $EndComp
@@
 	9550 1400 10000 1400
 Wire Wire Line
-	800  1000 1600 1000
+	600  1000 1600 1000
 Text Label 4100 7550 2    66   ~ 0
 RESET
@@
 	10550 3050 9950 3050
 Wire Wire Line
-	9950 3450 10550 3450
-Wire Wire Line
 	9950 3650 10550 3650
 Wire Wire Line
@@
 Text Label 4100 7450 2    70   ~ 0
 SCK
-Wire Wire Line
-	9950 3350 10550 3350
-Wire Wire Line
-	9950 3250 10550 3250
 Wire Wire Line
 	9950 3150 10550 3150
@@
 F 0 "R53" V 5725 2950 50  0000 C CNN
 F 1 "510" V 5800 2950 50  0000 C CNN
-F 2 "Resistor_SMD:R_0402_1005Metric" V 5730 2950 50  0001 C CNN
+F 2 "Resistor_SMD:R_0603_1608Metric_Pad0.98x0.95mm_HandSolder" V 5730 2950 50  0001 C CNN
 F 3 "~" H 5800 2950 50  0001 C CNN
 	1    5800 2950
@@
 F 0 "R56" V 5725 2750 50  0000 C CNN
 F 1 "510" V 5800 2750 50  0000 C CNN
-F 2 "Resistor_SMD:R_0402_1005Metric" V 5730 2750 50  0001 C CNN
+F 2 "Resistor_SMD:R_0603_1608Metric_Pad0.98x0.95mm_HandSolder" V 5730 2750 50  0001 C CNN
 F 3 "~" H 5800 2750 50  0001 C CNN
 	1    5800 2750
@@
 F 0 "R52" V 5725 2550 50  0000 C CNN
 F 1 "510" V 5800 2550 50  0000 C CNN
-F 2 "Resistor_SMD:R_0402_1005Metric" V 5730 2550 50  0001 C CNN
+F 2 "Resistor_SMD:R_0603_1608Metric_Pad0.98x0.95mm_HandSolder" V 5730 2550 50  0001 C CNN
 F 3 "~" H 5800 2550 50  0001 C CNN
 	1    5800 2550
@@
 F 0 "R49" V 5725 2350 50  0000 C CNN
 F 1 "510" V 5800 2350 50  0000 C CNN
-F 2 "Resistor_SMD:R_0402_1005Metric" V 5730 2350 50  0001 C CNN
+F 2 "Resistor_SMD:R_0603_1608Metric_Pad0.98x0.95mm_HandSolder" V 5730 2350 50  0001 C CNN
 F 3 "~" H 5800 2350 50  0001 C CNN
 	1    5800 2350
@@
 	5550 2550 5650 2550
 NoConn ~ 1600 800
+Text Label 9850 3350 2    50   ~ 0
+SDI
+Text Label 9850 3450 2    50   ~ 0
+SEN
+Text Label 9850 3250 2    50   ~ 0
+SDO
+Wire Wire Line
+	9850 3350 10550 3350
+Wire Wire Line
+	9850 3450 10550 3450
+Wire Wire Line
+	9850 3250 10550 3250
+NoConn ~ 600  1100
+Text Label 1450 1500 0    70   ~ 0
+VIN
+Wire Wire Line
+	1450 1500 1600 1500
+$Comp
+L power:VDDA #PWR0141
+U 1 1 6100AC4A
+P 1100 1500
+F 0 "#PWR0141" H 1100 1350 50  0001 C CNN
+F 1 "VDDA" V 1100 1700 50  0000 C CNN
+F 2 "" H 1100 1500 50  0001 C CNN
+F 3 "" H 1100 1500 50  0001 C CNN
+	1    1100 1500
+	0    -1   -1   0
+$EndComp
+Wire Wire Line
+	1100 1500 1150 1500
+$Comp
+L Device:R R100
+U 1 1 61018AD7
+P 1300 1500
+F 0 "R100" V 1400 1500 50  0000 C CNN
+F 1 "0" V 1300 1500 50  0000 C CNN
+F 2 "Resistor_SMD:R_0603_1608Metric_Pad0.98x0.95mm_HandSolder" V 1230 1500 50  0001 C CNN
+F 3 "~" H 1300 1500 50  0001 C CNN
+	1    1300 1500
+	0    1    1    0
+$EndComp
+NoConn ~ 9550 1200
+NoConn ~ 9550 1300
+NoConn ~ 9550 1400
+NoConn ~ 10700 1300
+NoConn ~ 600  5700
+NoConn ~ 600  5800
+NoConn ~ 600  5900
+NoConn ~ 600  6000
+NoConn ~ 10050 5500
+NoConn ~ 10050 5600
+NoConn ~ 10050 5700
+NoConn ~ 10050 5800
+NoConn ~ 10050 5900
+NoConn ~ 10050 6000
+NoConn ~ 10050 6100
+NoConn ~ 10050 6200
+NoConn ~ 9950 2950
+NoConn ~ 9950 3550
+NoConn ~ 9950 3650
+Text Label 600  1200 0    21   ~ 0
++5V_Ard
+$Comp
+L power:PWR_FLAG #FLG0108
+U 1 1 61B189E4
+P 1350 3650
+F 0 "#FLG0108" H 1350 3725 50  0001 C CNN
+F 1 "PWR_FLAG" H 1350 3823 50  0000 C CNN
+F 2 "" H 1350 3650 50  0001 C CNN
+F 3 "~" H 1350 3650 50  0001 C CNN
+	1    1350 3650
+	1    0    0    -1
+$EndComp
+Wire Wire Line
+	1100 3400 1100 3250
+$Comp
+L Connector:Barrel_Jack_Switch J?
+U 1 1 610E86EA
+P 750 3500
+F 0 "J?" H 807 3817 50  0000 C CNN
+F 1 "Barrel_Jack_Switch" H 807 3726 50  0000 C CNN
+F 2 "" H 800 3460 50  0001 C CNN
+F 3 "~" H 800 3460 50  0001 C CNN
+	1    750  3500
+	1    0    0    -1
+$EndComp
+Wire Wire Line
+	1050 3400 1100 3400
+Wire Wire Line
+	1050 3500 1100 3500
+Wire Wire Line
+	1100 3500 1100 3600
+Wire Wire Line
+	1050 3600 1100 3600
+Connection ~ 1100 3600
+Wire Wire Line
+	1100 3600 1100 3750
 $EndSCHEMATC
