File: AD9851.kicad_sch (KiCad schematic)
At the start: 9 parts

Commit message: Added filters on output wired the option to have all of the amplifier parallel bits connected
Parts:
- C4, C6, C7: renamed from C?; footprint (none) -> Capacitor_SMD:C_0603_1608Metric_Pad1.08x0.95mm_HandSolder
- R26, R27, R28: renamed from R?; footprint (none) -> Resistor_SMD:R_0603_1608Metric_Pad0.98x0.95mm_HandSolder
- gave numbers to parts that had none: 3
Changed lines of the file:
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@@
   (symbol (lib_id "Device:C") (at 127 57.15 0) (unit 1)
     (in_bom yes) (on_board yes)
-    (property "Reference" "C?" (id 0) (at 128.27 54.61 0)
+    (property "Reference" "C6" (id 0) (at 128.27 54.61 0)
       (effects (font (size 1.27 1.27)) (justify left))
     )
@@
       (effects (font (size 1.27 1.27)) (justify left))
     )
-    (property "Footprint" "" (id 2) (at 127.9652 60.96 0)
+    (property "Footprint" "Capacitor_SMD:C_0603_1608Metric_Pad1.08x0.95mm_HandSolder" (id 2) (at 127.9652 60.96 0)
       (effects (font (size 1.27 1.27)) hide)
     )
@@
   (symbol (lib_id "power:VDD") (at 76.2 85.09 0) (unit 1)
     (in_bom yes) (on_board yes)
-    (property "Reference" "#PWR?" (id 0) (at 76.2 88.9 0)
+    (property "Reference" "#PWR0113" (id 0) (at 76.2 88.9 0)
       (effects (font (size 1.27 1.27)) hide)
     )
@@
   (symbol (lib_id "power:GND") (at 144.78 91.44 90) (unit 1)
     (in_bom yes) (on_board yes)
-    (property "Reference" "#PWR?" (id 0) (at 151.13 91.44 0)
+    (property "Reference" "#PWR0117" (id 0) (at 151.13 91.44 0)
       (effects (font (size 1.27 1.27)) hide)
     )
@@
   (symbol (lib_id "Device:C") (at 69.85 91.44 180) (unit 1)
     (in_bom yes) (on_board yes)
-    (property "Reference" "C?" (id 0) (at 70.485 89.535 0)
+    (property "Reference" "C10" (id 0) (at 70.485 89.535 0)
       (effects (font (size 1.27 1.27)) (justify right))
     )
@@
   (symbol (lib_id "power:GND") (at 127 63.5 0) (unit 1)
     (in_bom yes) (on_board yes)
-    (property "Reference" "#PWR?" (id 0) (at 127 69.85 0)
+    (property "Reference" "#PWR0116" (id 0) (at 127 69.85 0)
       (effects (font (size 1.27 1.27)) hide)
     )
@@
   (symbol (lib_id "power:GND") (at 69.85 96.52 0) (unit 1)
     (in_bom yes) (on_board yes)
-    (property "Reference" "#PWR?" (id 0) (at 69.85 102.87 0)
+    (property "Reference" "#PWR0108" (id 0) (at 69.85 102.87 0)
       (effects (font (size 1.27 1.27)) hide)
     )
@@
   (symbol (lib_id "power:VDD") (at 144.78 93.98 270) (unit 1)
     (in_bom yes) (on_board yes)
-    (property "Reference" "#PWR?" (id 0) (at 140.97 93.98 0)
+    (property "Reference" "#PWR0118" (id 0) (at 140.97 93.98 0)
       (effects (font (size 1.27 1.27)) hide)
     )
@@
   (symbol (lib_id "Device:R") (at 109.22 69.85 180) (unit 1)
     (in_bom yes) (on_board yes)
-    (property "Reference" "R?" (id 0) (at 107.188 69.85 90))
+    (property "Reference" "R27" (id 0) (at 107.188 69.85 90))
     (property "Value" "10k" (id 1) (at 109.22 69.85 90))
-    (property "Footprint" "" (id 2) (at 110.998 69.85 90)
+    (property "Footprint" "Resistor_SMD:R_0603_1608Metric_Pad0.98x0.95mm_HandSolder" (id 2) (at 110.998 69.85 90)
       (effects (font (size 1.27 1.27)) hide)
     )
@@
   (symbol (lib_id "power:VDD") (at 106.68 63.5 0) (unit 1)
     (in_bom yes) (on_board yes) (fields_autoplaced)
-    (property "Reference" "#PWR?" (id 0) (at 106.68 67.31 0)
+    (property "Reference" "#PWR0119" (id 0) (at 106.68 67.31 0)
       (effects (font (size 1.27 1.27)) hide)
     )
@@
   (symbol (lib_id "power:GND") (at 127 116.84 0) (unit 1)
     (in_bom yes) (on_board yes)
-    (property "Reference" "#PWR?" (id 0) (at 127 123.19 0)
+    (property "Reference" "#PWR0114" (id 0) (at 127 123.19 0)
       (effects (font (size 1.27 1.27)) hide)
     )
@@
   (symbol (lib_id "Device:R") (at 104.14 69.85 180) (unit 1)
     (in_bom yes) (on_board yes)
-    (property "Reference" "R?" (id 0) (at 102.108 69.85 90))
+    (property "Reference" "R26" (id 0) (at 102.108 69.85 90))
     (property "Value" "10k" (id 1) (at 104.14 69.85 90))
-    (property "Footprint" "" (id 2) (at 105.918 69.85 90)
+    (property "Footprint" "Resistor_SMD:R_0603_1608Metric_Pad0.98x0.95mm_HandSolder" (id 2) (at 105.918 69.85 90)
       (effects (font (size 1.27 1.27)) hide)
     )
@@
   (symbol (lib_id "power:GND") (at 153.67 107.95 0) (unit 1)
     (in_bom yes) (on_board yes)
-    (property "Reference" "#PWR?" (id 0) (at 153.67 114.3 0)
+    (property "Reference" "#PWR0115" (id 0) (at 153.67 114.3 0)
       (effects (font (size 1.27 1.27)) hide)
     )
@@
   (symbol (lib_id "Device:C") (at 119.38 57.15 0) (unit 1)
     (in_bom yes) (on_board yes)
-    (property "Reference" "C?" (id 0) (at 120.65 54.61 0)
+    (property "Reference" "C4" (id 0) (at 120.65 54.61 0)
       (effects (font (size 1.27 1.27)) (justify left))
     )
@@
       (effects (font (size 1.27 1.27)) (justify left))
     )
-    (property "Footprint" "" (id 2) (at 120.3452 60.96 0)
+    (property "Footprint" "Capacitor_SMD:C_0603_1608Metric_Pad1.08x0.95mm_HandSolder" (id 2) (at 120.3452 60.96 0)
       (effects (font (size 1.27 1.27)) hide)
     )
@@
   (symbol (lib_id "power:GND") (at 104.14 87.63 0) (unit 1)
     (in_bom yes) (on_board yes)
-    (property "Reference" "#PWR?" (id 0) (at 104.14 93.98 0)
+    (property "Reference" "#PWR0112" (id 0) (at 104.14 93.98 0)
       (effects (font (size 1.27 1.27)) hide)
     )
@@
   (symbol (lib_id "power:VDD") (at 127 50.8 0) (unit 1)
     (in_bom yes) (on_board yes) (fields_autoplaced)
-    (property "Reference" "#PWR?" (id 0) (at 127 54.61 0)
+    (property "Reference" "#PWR0120" (id 0) (at 127 54.61 0)
       (effects (font (size 1.27 1.27)) hide)
     )
@@
   (symbol (lib_id "Interface:AD9851") (at 127 91.44 0) (unit 1)
     (in_bom yes) (on_board yes) (fields_autoplaced)
-    (property "Reference" "U?" (id 0) (at 131.5594 68.58 0)
+    (property "Reference" "U2" (id 0) (at 131.5594 68.58 0)
       (effects (font (size 1.27 1.27)) (justify left))
     )
@@
   (symbol (lib_id "Device:R") (at 148.59 106.68 90) (unit 1)
     (in_bom yes) (on_board yes)
-    (property "Reference" "R?" (id 0) (at 148.59 104.648 90))
+    (property "Reference" "R28" (id 0) (at 148.59 104.648 90))
     (property "Value" "3.9k" (id 1) (at 148.59 106.68 90))
-    (property "Footprint" "" (id 2) (at 148.59 108.458 90)
+    (property "Footprint" "Resistor_SMD:R_0603_1608Metric_Pad0.98x0.95mm_HandSolder" (id 2) (at 148.59 108.458 90)
       (effects (font (size 1.27 1.27)) hide)
     )
@@
   (symbol (lib_id "power:GND") (at 76.2 119.38 0) (unit 1)
     (in_bom yes) (on_board yes)
-    (property "Reference" "#PWR?" (id 0) (at 76.2 125.73 0)
+    (property "Reference" "#PWR0109" (id 0) (at 76.2 125.73 0)
       (effects (font (size 1.27 1.27)) hide)
     )
@@
   (symbol (lib_id "Oscillator:ASV-xxxMHz") (at 76.2 109.22 0) (unit 1)
     (in_bom yes) (on_board yes)
-    (property "Reference" "X?" (id 0) (at 80.01 102.87 0))
+    (property "Reference" "X1" (id 0) (at 80.01 102.87 0))
     (property "Value" "ASV-30MHz" (id 1) (at 82.55 116.84 0))
     (property "Footprint" "Oscillator:Oscillator_SMD_Abracon_ASV-4Pin_7.0x5.1mm" (id 2) (at 93.98 118.11 0)
@@
   (symbol (lib_id "Device:C") (at 134.62 57.15 0) (unit 1)
     (in_bom yes) (on_board yes)
-    (property "Reference" "C?" (id 0) (at 135.89 54.61 0)
+    (property "Reference" "C7" (id 0) (at 135.89 54.61 0)
       (effects (font (size 1.27 1.27)) (justify left))
     )
@@
       (effects (font (size 1.27 1.27)) (justify left))
     )
-    (property "Footprint" "" (id 2) (at 135.5852 60.96 0)
-      (effects (font (size 1.27 1.27)) hide)
-    )
+    (property "Footprint" "Capacitor_SMD:C_0603_1608Metric_Pad1.08x0.95mm_HandSolder" (id 2) (at 135.5852 60.96 0)
+      (effects (font (size 1.27 1.27)) hide)
+    )
